File: GBDSO-Modules.sch (KiCad schematic (older format))
At the start: 75 parts, among them J1 MJ-3523-SMT-TR, J2 MJ-3523-SMT-TR, J3 EdgeConnector, J5 Conn_01x02, J6 Conn_01x02, P1 100k, P2 100k, SW1 SW_SPDT, SW2 SW_SPDT, U1 TL072, U2 DS1267_SOIC, U3 TL072, U4 MAX114CAG, U5 74HC175D, U6 74HC138D, U7 AT27C256R, U8 TLC272, U9 MAX828

Commit message: separated each module into a different sheet, started the pcb
Parts:
- removed C1, C10: 18p, Capacitor_SMD:C_0805_2012Metric, symbol Device:C_Small
- removed C11, C12, C14, C17, C18, C19, C2, C20, C21, C23, C27, C29, C30, C4, C5, C8, C9: 100n, Capacitor_SMD:C_0805_2012Metric, symbol Device:C_Small
- removed C13, C3: 1p8, Capacitor_SMD:C_0805_2012Metric, symbol Device:C_Small
- removed C15, C6: 15p, Capacitor_SMD:C_0805_2012Metric, symbol Device:C_Small
- removed C16, C7: 220p, Capacitor_SMD:C_0805_2012Metric, symbol Device:C_Small
- removed C22, C24, C25, C26, C28, C31, C33: 10µ, Capacitor_SMD:C_1206_3216Metric, symbol Device:CP1_Small
- removed D1, D2: BAV199, Package_TO_SOT_SMD:SOT-23_Handsoldering, symbol BAV199:BAV199
- removed D3: ZR4040-2.5, Package_TO_SOT_SMD:SOT-23_Handsoldering, symbol ZR40402F25TA:ZR4040-2.5
- removed J1, J2: MJ-3523-SMT-TR, MJ-3523-SMT-TR:MJ-3523-SMT-TR, symbol MJ-3523-SMT-TR:MJ-3523-SMT-TR
- removed J3: EdgeConnector, GB_EdgeConnector:GB_EdgeConnector, symbol Connector_Generic:Conn_01x32
- removed J5, J6: Conn_01x02, Connector_PinHeader_2.54mm:PinHeader_1x02_P2.54mm_Horizontal, symbol Connector_Generic:Conn_01x02
- removed JP1: SolderJumper_3_Open, Jumper:SolderJumper-3_P1.3mm_Open_RoundedPad1.0x1.5mm_NumberLabels, symbol Jumper:SolderJumper_3_Open
- removed JP2: SolderJumper_2_Open, Jumper:SolderJumper-2_P1.3mm_Open_TrianglePad1.0x1.5mm, symbol Jumper:SolderJumper_2_Open
- removed L1, L2, L3: 100µ, Inductor_SMD:L_0805_2012Metric_Pad1.15x1.40mm_HandSolder, symbol Device:L_Small
- removed P1, P2: 100k, Potentiometer_SMD:Potentiometer_Vishay_TS53YJ_Vertical, symbol Device:R_POT_TRIM
- removed R1, R11, R2, R4, R8, R9: 1M, Resistor_SMD:R_0805_2012Metric, symbol Device:R
- removed R10, R13, R14, R3, R6, R7: 4k7, Resistor_SMD:R_0805_2012Metric, symbol Device:R
- removed R12, R5: 470k, Resistor_SMD:R_0805_2012Metric, symbol Device:R
- removed R15: 15k, Resistor_SMD:R_0805_2012Metric, symbol Device:R
- removed R16, R17: 100k, Resistor_SMD:R_0805_2012Metric, symbol Device:R
- removed SW1, SW2: SW_SPDT, Button_Switch_SMD:SW_SPDT_CK-JS102011SAQN, symbol Switch:SW_SPDT
- removed U1, U3: TL072, Package_SO:SOIC-8_3.9x4.9mm_P1.27mm, symbol Amplifier_Operational:TL072
- removed U2: DS1267_SOIC, Package_SO:SOIC-16W_7.5x10.3mm_P1.27mm, symbol Potentiometer_Digital:DS1267_SOIC
- removed U4: MAX114CAG, Package_SO:SSOP-24_5.3x8.2mm_P0.65mm, symbol MAX114CAG:MAX114CAG
- removed U5: 74HC175D, Package_SO:SOIC-16_3.9x9.9mm_P1.27mm, symbol 74HC175D:74HC175D
- removed U6: 74HC138D, Package_SO:SOIC-16_3.9x9.9mm_P1.27mm, symbol 74HC138D:74HC138D
- removed U7: AT27C256R, Package_LCC:PLCC-32_11.4x14.0mm_P1.27mm, symbol AT27C256R:AT27C256R
- removed U8: TLC272, Package_SO:SOIC-8_3.9x4.9mm_P1.27mm, symbol Amplifier_Operational:TLC272
- removed U9: MAX828, Package_TO_SOT_SMD:SOT-23-5_HandSoldering, symbol MAX828EUK:MAX828
Connections:
- net labels removed: +2.5V, +5V, +5VA, +5VC, -2.5V, -5V, A0, A1, A10, A11, A12, A13, A14, A15, A2, A3, A4, A5, A6, A7, A8, A9, D0, D1, D2, D3, D4, D5, D6, D7, ECLK, GND, VPP, ~RD, ~WR
- wire segments 423 -> 0
- no-connect marks 19 -> 0
Other:
- note removed: "CH A"
- note removed: "CH B"
