File: 2V5 Gen.sch (KiCad schematic (older format))
At the start: 9 parts, among them J19 Conn_01x06, U8 TLC272

Commit message: fixed schematic and updated PCB
Fixed the schematic after having found the issues in the GBDSO schematic (which is also fixed on the repo).
Continued making the PCB for the modules. We're not at 7 modules from 10.
Parts:
- J19: footprint Package_DIP:DIP-6_W7.62mm -> Package_DIP:DIP-6_W10.16mm
Changed lines of the file:
@@
 F 0 "J19" H 3670 2752 50  0000 L CNN
 F 1 "Conn_01x06" H 3670 2661 50  0000 L CNN
-F 2 "Package_DIP:DIP-6_W7.62mm" H 3590 2760 50  0001 C CNN
+F 2 "Package_DIP:DIP-6_W10.16mm" H 3590 2760 50  0001 C CNN
 F 3 "~" H 3590 2760 50  0001 C CNN
 	1    3590 2760
