File: DFF.sch (KiCad schematic (older format))
At the start: 3 parts, among them J14 Conn_01x12, U5 74HC175D

Commit message: fixed schematic and updated PCB
Fixed the schematic after having found the issues in the GBDSO schematic (which is also fixed on the repo).
Continued making the PCB for the modules. We're not at 7 modules from 10.
Parts:
- J14: footprint Package_DIP:DIP-12_W7.62mm -> Package_DIP:DIP-12_W10.16mm_LongPads
Changed lines of the file:
@@
 F 0 "J14" H 4100 1652 50  0000 L CNN
 F 1 "Conn_01x12" H 4100 1561 50  0000 L CNN
-F 2 "Package_DIP:DIP-12_W7.62mm" H 4020 1660 50  0001 C CNN
+F 2 "Package_DIP:DIP-12_W10.16mm_LongPads" H 4020 1660 50  0001 C CNN
 F 3 "~" H 4020 1660 50  0001 C CNN
 	1    4020 1660
