File: OTP ROM.sch (KiCad schematic (older format))
At the start: 4 parts, among them J16 Conn_01x28, U7 AT27C256R

Commit message: added the PLCC32 handsolder footprint I made on the other repo here
Parts:
- U7: footprint Package_LCC:PLCC-32_11.4x14.0mm_P1.27mm -> PLCC32_HandSolder:PLCC-32_HandSolder
Changed lines of the file:
@@
 F 0 "U7" H 1440 3200 50  0000 C CNN
 F 1 "AT27C256R" H 1990 3200 50  0000 C CNN
-F 2 "Package_LCC:PLCC-32_11.4x14.0mm_P1.27mm" H 2640 1450 50  0001 C CNN
+F 2 "PLCC32_HandSolder:PLCC-32_HandSolder" H 2640 1450 50  0001 C CNN
 F 3 "" H 1690 2350 50  0001 C CNN
 	1    1690 2350
