File: Digital Pot.sch (KiCad schematic (older format))
At the start: 4 parts, among them J12 Conn_01x12, U2 DS1267_SOIC

Commit message: C8 on the dig pot wasn't connected correctly
changed the schematic, updated the netlist and PCB
Connections:
- net -5V: no longer C8.2
- net GND: now also C8.2
Changed lines of the file:
@@
 Wire Wire Line
 	1550 2760 1550 2680
-Text GLabel 1550 2760 3    50   Input ~ 0
+Text GLabel 1480 2430 0    50   Input ~ 0
 -5V
 Wire Wire Line
@@
 	1750 2430 1550 2430
 Wire Wire Line
-	1850 2470 1850 2380
+	1850 2820 1850 2760
 $Comp
 L power:GND #PWR?
 U 1 1 5FAC0B85
-P 1850 2470
+P 1850 2820
 AR Path="/5F6C55C3/5FAC0B85" Ref="#PWR?"  Part="1"
 AR Path="/5FABC497/5FAC0B85" Ref="#PWR0121"  Part="1"
-F 0 "#PWR0121" H 1850 2220 50  0001 C CNN
-F 1 "GND" H 1855 2297 50  0000 C CNN
-F 2 "" H 1850 2470 50  0001 C CNN
-F 3 "" H 1850 2470 50  0001 C CNN
-	1    1850 2470
+F 0 "#PWR0121" H 1850 2570 50  0001 C CNN
+F 1 "GND" H 1855 2647 50  0000 C CNN
+F 2 "" H 1850 2820 50  0001 C CNN
+F 3 "" H 1850 2820 50  0001 C CNN
+	1    1850 2820
 	1    0    0    -1
 $EndComp
@@
 Wire Wire Line
 	3990 1450 4020 1450
+Wire Wire Line
+	1550 2760 1850 2760
+Connection ~ 1850 2760
+Wire Wire Line
+	1850 2760 1850 2380
 $EndSCHEMATC

Commit message: pin 10 of J12 was not connected to the correct signal, fixed
Parts:
- J12: footprint Package_DIP:DIP-12_W7.62mm -> Connector_PinHeader_2.54mm:PinHeader_1x12_P2.54mm_Vertical
Connections:
- net -5V: now also C8.1, U2.1 (VB)
- net DPOT_0H: no longer J12.10 (Pin_10)
- net DPOT_1H: now also J12.10 (Pin_10)
Changed lines of the file:
@@
 F 0 "J12" H 4300 1642 50  0000 L CNN
 F 1 "Conn_01x12" H 4300 1551 50  0000 L CNN
-F 2 "Package_DIP:DIP-12_W7.62mm" H 4220 1650 50  0001 C CNN
+F 2 "Connector_PinHeader_2.54mm:PinHeader_1x12_P2.54mm_Vertical" H 4220 1650 50  0001 C CNN
 F 3 "~" H 4220 1650 50  0001 C CNN
 	1    4220 1650
@@
 DPOT_1W
 Text GLabel 3990 2050 0    50   Output ~ 0
-DPOT_0H
+DPOT_1H
 Text GLabel 3990 1450 0    50   Output ~ 0
 D1
@@
 Wire Wire Line
 	1850 2760 1850 2380
+Wire Wire Line
+	1480 2430 1550 2430
+Connection ~ 1550 2430
 $EndSCHEMATC
